File: ContactorDriver.kicad_sch (KiCad schematic)
At the start: 49 parts, among them J1 PowerConn, J10 FanConn3, J11 FanConn4, J12 ContactorAConn, J2 DashboardConnA, J3 ContactorBConn, J4 DashboardConnB, J5 ContactorCConn, J6 DashboardConnC, J8 FanConn1, J9 FanConn2, Q1 PMV35EPER, Q2 IRLML0030TRPbF, Q3 IRLML0030TRPbF, Q4 IRLML0030TRPbF, U1 SFH617A-1, U2 SFH617A-1, U3 SFH617A-1

Commit message: small layout/silkscreen changes and finalizing
Other:
- note added: "Auxilary pins sent back to Controls to see Contactor status"
- note added: "Contactor Control"
- note added: "Sense Optoisolators"
- note added: "We pass our 12V and Controls sends it back via an optoisolator once ready to close"
- note removed: "Precharge Contactor Control"
- moved on the sheet: R10, R11, R9, U1, U2, U3
